File: BenchBudEE/BenchBudEE.sch (KiCad schematic (older format))
At the start: 0 parts

Commit message: fan schematic
Changed lines of the file:
@@
 LIBS:contrib
 LIBS:valves
+LIBS:BenchBudEE-cache
 EELAYER 27 0
 EELAYER END
@@
 Sheet 1 8
 Title ""
-Date "6 feb 2014"
+Date "8 feb 2014"
 Rev ""
 Comp ""
@@
 $EndSheet
 $Sheet
-S 7450 1800 1000 1000
-U 52F19A3C
-F0 "Fan" 50
-F1 "fan.sch" 50
-F2 "POWER+" O R 8450 2000 60
-F3 "POWER-" I R 8450 2200 60
-F4 "TACH_IN" I R 8450 2400 60
-F5 "TACH_OUT" O L 7450 2100 60
-F6 "FAN_IN" I L 7450 2300 60
-$EndSheet
-$Sheet
 S 7400 4550 1100 1050
 U 52F19A48
@@
 F4 "SCLK" I L 7400 3750 60
 F5 "~CS" I L 7400 3950 60
-F6 "TC_IN+" I R 8500 3400 60
-F7 "TC_IN-" I R 8500 3600 60
+F6 "TC_IN+" I R 8500 3350 60
+F7 "TC_IN-" I R 8500 3550 60
 $EndSheet
 $Sheet
-S 7400 5850 1150 1050
+S 7400 5850 1100 1050
 U 52F19A58
 F0 "Relay" 50
@@
 F2 "D_IN+" I L 7400 6050 60
 F3 "D_IN-" I L 7400 6250 60
-F4 "RELAY+" O R 8550 6050 60
-F5 "RELAY-" I R 8550 6250 60
+F4 "RELAY+" O R 8500 6050 60
+F5 "RELAY-" I R 8500 6250 60
+$EndSheet
+$Sheet
+S 7400 1000 1100 1500
+U 52F19A3C
+F0 "Fan" 50
+F1 "fan.sch" 50
+F2 "POWER+" O R 8500 1150 60
+F3 "POWER-" I R 8500 1300 60
+F4 "TACH_IN" I R 8500 1450 60
+F5 "TACH_OUT" O L 7400 2400 60
+F6 "FAN_IN" I L 7400 1150 60
+F7 "Current_Measure" O L 7400 2250 60
+F8 "MOSI" I L 7400 1750 60
+F9 "MISO" O L 7400 1850 60
+F10 "~CS" I L 7400 1950 60
+F11 "SCLK" I L 7400 2050 60
 $EndSheet
 $EndSCHEMATC
