File: BenchBudEE/BenchBudEE.sch (KiCad schematic (older format))
At the start: 0 parts

Commit message: power schematic
Changed lines of the file:
@@
 $Descr A4 11693 8268
 encoding utf-8
-Sheet 1 8
+Sheet 1 9
 Title ""
-Date "8 feb 2014"
+Date "12 feb 2014"
 Rev ""
 Comp ""
@@
 $EndSheet
 $Sheet
-S 3350 2600 1000 1000
+S 1750 1700 1000 1000
 U 52F19A2E
 F0 "Power" 50
@@
 F11 "SCLK" I L 7400 2050 60
 $EndSheet
+$Sheet
+S 4550 1650 1550 1050
+U 52FADC37
+F0 "PowerAdjustmentMonitor" 50
+F1 "PowerAdjustmentMonitor.sch" 50
+$EndSheet
 $EndSCHEMATC
