File: BenchBudEE/fan.sch (KiCad schematic (older format))
At the start: 0 parts

Commit message: fan schematic
Parts:
- added Q?: MOSFET_N, ~, symbol MOSFET_N
- added R? (x4): R, ~, symbol R
- added RV?: POT, ~, symbol POT
- added U?: LM324, symbol LM324
- added U?: MCP4922-E/P, DIP14, symbol MCP4922-E/P
Connections:
- net FAN_IN: now also R?.2, R?.2
- net POWER+: now also Q?.S
- new net: Q?.G, U?.1
- new net: R?.2, RV?.3, U?.14 (VoutA), U?.3 (+)
- new net: R?.1, U?.9 (~SHDN~)
- new net +12V: Q?.D, R?.1, U?.4 (V+)
- new net -12V: U?.11 (V-)
- new net AGND: R?.2, RV?.1
- new net Current_Measure: R?.1, R?.1, U?.2 (-)
- new net MOSI: U?.5 (SDI)
- new net SCLK: U?.4 (SCK)
- new net ~CS: U?.3 (~CS~)
