File: BenchBudEE/relay.sch (KiCad schematic (older format))
At the start: 0 parts

Commit message: relay schematic
Parts:
- added D?: LED, ~, symbol LED
- added D?: DIODE, ~, symbol DIODE
- added K?: RELAY_SPDT, ~, symbol RELAY_SPDT
- added Q?: NPN, ~, symbol NPN
- added R? (x6): R, ~, symbol R
- added U?: PHTRANS, ~, symbol PHTRANS
Connections:
- net labels added: +12V, COM, GND, NC, NO
- net labels removed: RELAY+, RELAY-
- wire segments 0 -> 24
Changed lines of the file:
@@
 LIBS:contrib
 LIBS:valves
+LIBS:BenchBuddEE
 LIBS:BenchBudEE-cache
 EELAYER 27 0
@@
 $Descr A4 11693 8268
 encoding utf-8
-Sheet 8 8
+Sheet 7 8
 Title ""
 Date "8 feb 2014"
@@
 Comment4 ""
 $EndDescr
-Text HLabel 2250 2400 0    60   Input ~ 0
+Text HLabel 3600 3200 0    60   Input ~ 0
 D_IN+
-Text HLabel 2200 2900 0    60   Input ~ 0
+Text HLabel 3600 3550 0    60   Input ~ 0
 D_IN-
-Text HLabel 9450 2400 2    60   Output ~ 0
-RELAY+
-Text HLabel 9450 2950 2    60   Input ~ 0
-RELAY-
+Text HLabel 9950 2700 2    60   BiDi ~ 0
+NC
+Text HLabel 9950 2900 2    60   BiDi ~ 0
+NO
+$Comp
+L PHTRANS U?
+U 1 1 52F6CFE1
+P 5250 3400
+F 0 "U?" H 5200 3750 70  0000 C CNN
+F 1 "PHTRANS" H 5200 3050 70  0000 C CNN
+F 2 "~" H 5250 3400 60  0000 C CNN
+F 3 "~" H 5250 3400 60  0000 C CNN
+	1    5250 3400
+	1    0    0    -1
+$EndComp
+$Comp
+L R R?
+U 1 1 52F6CFFF
+P 6550 3600
+F 0 "R?" V 6630 3600 40  0000 C CNN
+F 1 "R" V 6557 3601 40  0000 C CNN
+F 2 "~" V 6480 3600 30  0000 C CNN
+F 3 "~" H 6550 3600 30  0000 C CNN
+	1    6550 3600
+	0    -1   -1   0
+$EndComp
+$Comp
+L NPN Q?
+U 1 1 52F6D00E
+P 8250 3600
+F 0 "Q?" H 8250 3450 50  0000 R CNN
+F 1 "NPN" H 8250 3750 50  0000 R CNN
+F 2 "~" H 8250 3600 60  0000 C CNN
+F 3 "~" H 8250 3600 60  0000 C CNN
+	1    8250 3600
+	1    0    0    -1
+$EndComp
+$Comp
+L LED D?
+U 1 1 52F6D01D
+P 6100 4000
+F 0 "D?" H 6100 4100 50  0000 C CNN
+F 1 "LED" H 6100 3900 50  0000 C CNN
+F 2 "~" H 6100 4000 60  0000 C CNN
+F 3 "~" H 6100 4000 60  0000 C CNN
+	1    6100 4000
+	0    1    1    0
+$EndComp
+$Comp
+L RELAY_SPDT K?
+U 1 1 52F6D612
+P 9200 2900
+F 0 "K?" H 9200 3350 70  0000 C CNN
+F 1 "RELAY_SPDT" H 9500 2450 70  0000 C CNN
+F 2 "~" H 9200 3050 60  0000 C CNN
+F 3 "~" H 9200 3050 60  0000 C CNN
+	1    9200 2900
+	1    0    0    -1
+$EndComp
+Text HLabel 8450 2800 0    60   BiDi ~ 0
+COM
+Wire Wire Line
+	8450 2800 8800 2800
+Wire Wire Line
+	9950 2900 9600 2900
+Wire Wire Line
+	9950 2700 9600 2700
+Wire Wire Line
+	6800 3600 8050 3600
+Wire Wire Line
+	8350 3400 8350 3100
+Wire Wire Line
+	8350 3100 8800 3100
+$Comp
+L +12V #PWR?
+U 1 1 52F6D670
+P 6800 2250
+F 0 "#PWR?" H 6800 2200 20  0001 C CNN
+F 1 "+12V" H 6800 2350 30  0000 C CNN
+F 2 "" H 6800 2250 60  0000 C CNN
+F 3 "" H 6800 2250 60  0000 C CNN
+	1    6800 2250
+	1    0    0    -1
+$EndComp
+Wire Wire Line
+	6800 3000 8800 3000
+Wire Wire Line
+	4700 3200 3600 3200
+Wire Wire Line
+	5850 3600 6300 3600
+Wire Wire Line
+	6800 3400 5800 3400
+Wire Wire Line
+	8350 4000 8350 3800
+$Comp
+L R R?
+U 1 1 52F6D6E2
+P 8350 4250
+F 0 "R?" V 8430 4250 40  0000 C CNN
+F 1 "R" V 8357 4251 40  0000 C CNN
+F 2 "~" V 8280 4250 30  0000 C CNN
+F 3 "~" H 8350 4250 30  0000 C CNN
+	1    8350 4250
+	-1   0    0    1
+$EndComp
+$Comp
+L GND #PWR?
+U 1 1 52F6D6EA
+P 8350 4700
+F 0 "#PWR?" H 8350 4700 30  0001 C CNN
+F 1 "GND" H 8350 4630 30  0001 C CNN
+F 2 "" H 8350 4700 60  0000 C CNN
+F 3 "" H 8350 4700 60  0000 C CNN
+	1    8350 4700
+	1    0    0    -1
+$EndComp
+Wire Wire Line
+	8350 4700 8350 4500
+$Comp
+L R R?
+U 1 1 52F6D710
+P 6100 4650
+F 0 "R?" V 6180 4650 40  0000 C CNN
+F 1 "R" V 6107 4651 40  0000 C CNN
+F 2 "~" V 6030 4650 30  0000 C CNN
+F 3 "~" H 6100 4650 30  0000 C CNN
+	1    6100 4650
+	-1   0    0    1
+$EndComp
+Wire Wire Line
+	6100 4400 6100 4200
+Wire Wire Line
+	6100 3800 6100 3600
+Connection ~ 6100 3600
+$Comp
+L GND #PWR?
+U 1 1 52F6D737
+P 6100 5100
+F 0 "#PWR?" H 6100 5100 30  0001 C CNN
+F 1 "GND" H 6100 5030 30  0001 C CNN
+F 2 "" H 6100 5100 60  0000 C CNN
+F 3 "" H 6100 5100 60  0000 C CNN
+	1    6100 5100
+	1    0    0    -1
+$EndComp
+Wire Wire Line
+	6100 5100 6100 4900
+$Comp
+L R R?
+U 1 1 52F6D75A
+P 6800 2650
+F 0 "R?" V 6880 2650 40  0000 C CNN
+F 1 "R" V 6807 2651 40  0000 C CNN
+F 2 "~" V 6730 2650 30  0000 C CNN
+F 3 "~" H 6800 2650 30  0000 C CNN
+	1    6800 2650
+	-1   0    0    1
+$EndComp
+Wire Wire Line
+	6800 2900 6800 3400
+Wire Wire Line
+	6800 2400 6800 2250
+Connection ~ 6800 3000
+$Comp
+L R R?
+U 1 1 52F6D79E
+P 6250 3200
+F 0 "R?" V 6330 3200 40  0000 C CNN
+F 1 "R" V 6257 3201 40  0000 C CNN
+F 2 "~" V 6180 3200 30  0000 C CNN
+F 3 "~" H 6250 3200 30  0000 C CNN
+	1    6250 3200
+	0    -1   -1   0
+$EndComp
+Wire Wire Line
+	6000 3200 5800 3200
+Wire Wire Line
+	6500 3200 6800 3200
+Connection ~ 6800 3200
+$Comp
+L R R?
+U 1 1 52F6D80B
+P 4150 3550
+F 0 "R?" V 4230 3550 40  0000 C CNN
+F 1 "R" V 4157 3551 40  0000 C CNN
+F 2 "~" V 4080 3550 30  0000 C CNN
+F 3 "~" H 4150 3550 30  0000 C CNN
+	1    4150 3550
+	0    -1   -1   0
+$EndComp
+Wire Wire Line
+	3900 3550 3600 3550
+Wire Wire Line
+	4400 3550 4700 3550
+$Comp
+L DIODE D?
+U 1 1 52F6D84F
+P 7950 3200
+F 0 "D?" H 7950 3300 40  0000 C CNN
+F 1 "DIODE" H 7950 3100 40  0000 C CNN
+F 2 "~" H 7950 3200 60  0000 C CNN
+F 3 "~" H 7950 3200 60  0000 C CNN
+	1    7950 3200
+	-1   0    0    1
+$EndComp
+Wire Wire Line
+	8150 3200 8350 3200
+Connection ~ 8350 3200
+Wire Wire Line
+	7750 3200 7600 3200
+Wire Wire Line
+	7600 3200 7600 3000
+Connection ~ 7600 3000
 $EndSCHEMATC

Commit message: power schematic
Connections:
- net labels added: +12P
- net labels removed: +12V
Changed lines of the file:
@@
 $Descr A4 11693 8268
 encoding utf-8
-Sheet 7 8
+Sheet 7 9
 Title ""
-Date "8 feb 2014"
+Date "12 feb 2014"
 Rev ""
 Comp ""
@@
 Wire Wire Line
 	8350 3100 8800 3100
-$Comp
-L +12V #PWR?
-U 1 1 52F6D670
-P 6800 2250
-F 0 "#PWR?" H 6800 2200 20  0001 C CNN
-F 1 "+12V" H 6800 2350 30  0000 C CNN
-F 2 "" H 6800 2250 60  0000 C CNN
-F 3 "" H 6800 2250 60  0000 C CNN
-	1    6800 2250
-	1    0    0    -1
-$EndComp
 Wire Wire Line
 	6800 3000 8800 3000
@@
 	7600 3200 7600 3000
 Connection ~ 7600 3000
+$Comp
+L +12P #PWR?
+U 1 1 52FAD9B8
+P 6800 2250
+F 0 "#PWR?" H 6800 2220 30  0001 C CNN
+F 1 "+12P" H 6800 2350 30  0000 C CNN
+F 2 "" H 6800 2250 60  0000 C CNN
+F 3 "" H 6800 2250 60  0000 C CNN
+	1    6800 2250
+	1    0    0    -1
+$EndComp
 $EndSCHEMATC
