File: BenchBudEE/relay.sch (KiCad schematic (older format))
At the start: 11 parts

Commit message: arduino schematic and interconnection
Connections:
- net labels added: RELAY+, RELAY-
- net labels removed: D_IN+, D_IN-
Changed lines of the file:
@@
 $Descr A4 11693 8268
 encoding utf-8
-Sheet 7 9
+Sheet 6 9
 Title ""
-Date "16 feb 2014"
+Date "17 feb 2014"
 Rev ""
 Comp ""
@@
 $EndDescr
 Text HLabel 3600 3200 0    60   Input ~ 0
-D_IN+
+RELAY+
 Text HLabel 3600 3550 0    60   Input ~ 0
-D_IN-
+RELAY-
 Text HLabel 9950 2700 2    60   BiDi ~ 0
 NC
